File: schematic/Water_Purifier.kicad_pcb (KiCad board)
At the start: 2 copper layers, 53.5 x 40.6 mm, 13 parts, among them J1 Conn_01x02_Female, J2 Conn_01x02_Female, Q1 IRLB8721PBF, U1 ATTINY85-20PU, U2 L7805CV

Commit message: final version + gerbers
Other:
- board text added: "+"
- board text added: "-"
- board text added: "Open Water v.1"
Changed lines of the file:
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@@
     (links 20)
     (no_connects 0)
-    (area 25.324999 23.462856 78.971345 68.755239)
+    (area 24.892 23.462856 78.994001 68.755239)
     (thickness 1.6)
-    (drawings 11)
+    (drawings 16)
     (tracks 62)
     (zones 0)
@@
     (visible_elements 7FFFFFFF)
     (pcbplotparams
-      (layerselection 0x00030_80000001)
-      (usegerberextensions false)
+      (layerselection 0x010f0_80000001)
+      (usegerberextensions true)
       (excludeedgelayer true)
       (linewidth 0.100000)
@@
       (outputformat 1)
       (mirror false)
-      (drillshape 1)
+      (drillshape 0)
       (scaleselection 1)
-      (outputdirectory ""))
+      (outputdirectory Gerbers/))
   )
   (net 0 "")
@@
       (effects (font (size 1 1) (thickness 0.15)) (justify mirror))
     )
-    (fp_text value JS202011SCQN (at 0.1 -5.575) (layer B.Fab)
-      (effects (font (size 1 1) (thickness 0.15)) (justify mirror))
+    (fp_text value JS202011SCQN (at 0.762 0.254) (layer F.SilkS)
+      (effects (font (size 1 1) (thickness 0.15)))
     )
     (fp_line (start -4.8 -4.25) (end 4.8 -4.25) (layer B.CrtYd) (width 0.05))
@@
       (net 8 GND))
   )
+  (gr_text "Open Water v.1" (at 59.944 27.432) (layer F.SilkS)
+    (effects (font (size 1.5 1.5) (thickness 0.3)))
+  )
+  (gr_text + (at 45.72 58.674) (layer F.SilkS)
+    (effects (font (size 1.5 1.5) (thickness 0.3)))
+  )
+  (gr_text - (at 43.18 58.674 90) (layer F.SilkS)
+    (effects (font (size 1.5 1.5) (thickness 0.3)))
+  )
+  (gr_text - (at 42.672 59.182) (layer F.Cu)
+    (effects (font (size 1.5 1.5) (thickness 0.3)))
+  )
+  (gr_text + (at 37.592 41.91) (layer F.SilkS)
+    (effects (font (size 1.5 1.5) (thickness 0.3)))
+  )
   (gr_text bulb (at 33.02 40.64 270) (layer F.SilkS)
